File: thunderbolt-gpu-adapter.kicad_sch (KiCad schematic)
At the start: 8 parts

Commit message: Fix PCIe power switch - layout, bump revision to 1.1.2
Other:
- company: (none) -> Antmicro Ltd
- title: (none) -> Thunderbolt GPU Adapter
Changed lines of the file:
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@@
   (paper "A3" portrait)
   (title_block
-    (date "2023-05-09")
-    (rev "1.1.1")
+    (title "Thunderbolt GPU Adapter")
+    (date "2023-11-21")
+    (rev "1.1.2")
+    (company "Antmicro Ltd")
     (comment 1 "www.antmicro.com")
-    (comment 2 "Antmicro Ltd.")
   )
   (image (at 146.685 98.425) (scale 3.5054)
@@
       (reference "U11") (unit 1) (value "AP22615A_TSOT26") (footprint "antmicro-footprints:TSOT23-6")
     )
-    (path "/c5be216d-0af2-4d3b-b234-e3e028a22446/feae62f1-4e4c-447c-9a8c-da62170a4a1f"
-      (reference "U12") (unit 1) (value "LT8350RV") (footprint "thunderbolt-gpu-adapter-footprints:QFN-32-4EP_4x6mm_P0.5mm")
-    )
     (path "/edaf7d73-1c1f-440c-ac8b-fe148d6370ed/b0a95c8b-a734-477e-a461-9131f29023c7"
