File: power.kicad_sch (KiCad schematic)
At the start: 158 parts, among them Q10 SI7613DN-T1-GE3, Q2 BC817-25W, Q3 DZDH0401DW, Q4 DZDH0401DW, Q5 SI7613DN-T1-GE3, Q6 SI7613DN-T1-GE3, Q8 BC817-25W, U1 LT8350RV#PBF, U10 LM3881MME_NOPB, U11 AP22615A_TSOT26, U2 MP2386GG, U3 TPS65983BAZBHR, U9 LM1117MP-3.3_NOPB

Commit message: Run kmake loclib
Parts:
- C131: footprint antmicro-footprints:C_0402_1005Metric -> thunderbolt-gpu-adapter-footprints:C_0402_1005Metric; symbol antmicroCapacitors0402:C_1u_0402 -> thunderbolt-gpu-adapter:C_1u_0402
- C132, C134: footprint antmicro-footprints:C_0603_1608Metric -> thunderbolt-gpu-adapter-footprints:C_0603_1608Metric; symbol antmicroCapacitors0603:C_10u_0603 -> thunderbolt-gpu-adapter:C_10u_0603
- R134: footprint antmicro-footprints:R_0402_1005Metric -> thunderbolt-gpu-adapter-footprints:R_0402_1005Metric; symbol antmicroResistors0402:R_2k2_0402 -> thunderbolt-gpu-adapter:R_2k2_0402
- U11: footprint antmicro-footprints:TSOT23-6 -> thunderbolt-gpu-adapter-footprints:TSOT23-6; symbol antmicroPMICPowerDistributionSwitchesLoadDrivers:AP22615A_TSOT26 -> thunderbolt-gpu-adapter:AP22615A_TSOT26

Commit message: Fix ERC errors on schematic:
	- Fix first batch of GND ERC
	- Fix second batch of GND ERC
	- Fix ERC of 0R_0603
	- Fix erc BC817-25W
	- Fix erc 220n_0402
	- Fix erc PCIe_x16_10146070-113Y0LF-vertical
	- Fix erc 100n_0402
	- Fix erc 10u_0805_35V
	- Correct BC817-25W_1
	- Correct erc R_98R_0402_1
	- Correct 10K_0402
	- Correct 22u/16V
	- Correct 100k
	- Correct 499R
	- Correct 3k01
	- Correct 10p
	- Correct 330R
	- Correct 3k3
	- Correct 1n4148WS-7-F
	- Correct SI7613DN-T1GE3_1 and TP's
	- Correct LED_G_0603_KP-1608CGCK_1
	- Correct 2k2_0402
	- Correct DZDH0401DW_1
	- Correct 22u_0603
	- Correct TP 0.75mm
	- Correct 0R_0402
	- Correct 0R_22.4A
	- Correct Batch of Resitors
	- Correct Batch of Capacitors
	- Correct USB PD controller
	- Correct batch of pasives
	- Correct MM3Z3V3C
	- Correct LM1117MP-3.3_NOPB
	- Correct Flash memory
	- Correct MP2386GG_1_1
	- Fix symbol LT8350RV#PBF and correct it on schematic
	- Add pwr flags
Parts:
- C119, C122, C38, C40, C42, C43, C46, C48, C50: Manufacturer Samsung -> Samsung Electro-Mechanics
- C16, C23, C27, C31, C39: Manufacturer Yaego -> YAGEO
- C33: MPN MC0402N330J500CT -> 04025A330FAT2A; Manufacturer Multicomp -> KYOCERA AVX
- C45, C49: MPN MC0402B221K500CT -> 04025C221JAT2A; Manufacturer Multicomp -> KYOCERA AVX
- Q3, Q4: MPN DZDH0401DW-7 -> DZDH0401DW
- R45: MPN WSLP1206R0200FEA -> WSLP1206R0200FEA
- R98, R99: Max. Curr. (none) -> 22.4A
- TP1, TP12, TP2, TP3, TP5, TP7, TP8: footprint thunderbolt-gpu-adapter-footprints:Testpoint_smd_1mm -> thunderbolt-gpu-adapter-footprints:TP_SMD_1mm
Other:
- moved on the sheet: C127, U9
